Commit message: init ICELED branch

File: amrROS2_ws/src/description/urdf/property/robot_property.urdf.xacro (robot description, xacro)
@@ -1,13 +1,13 @@
 <?xml version="1.0"?>
 <robot xmlns:xacro="http://ros.org/wiki/xacro">
-  <xacro:property name="base_length" value="0.5" />
-  <xacro:property name="base_width" value="0.44" />
-  <xacro:property name="base_height" value="0.22" />
+  <xacro:property name="base_length" value="0.48" />
+  <xacro:property name="base_width" value="0.42" />
+  <xacro:property name="base_height" value="0.24" />
   <xacro:property name="base_mass" value="30" />
-  <xacro:property name="wheel_radius" value="0.08255" />
-  <xacro:property name="wheel_width" value="0.047" />
+  <xacro:property name="wheel_radius" value="0.075" />
+  <xacro:property name="wheel_width" value="0.04" />
   <xacro:property name="wheel_pos_x" value="0.0" />
-  <xacro:property name="wheel_pos_y" value="0.1665" />
-  <xacro:property name="wheel_pos_z" value="-0.044" />
+  <xacro:property name="wheel_pos_y" value="0.168" />
+  <xacro:property name="wheel_pos_z" value="-0.115" />
   <xacro:property name="wheel_mass" value="1.236" />
   <xacro:property name="wheel_torque" value="20" />

File: amrROS2_ws/src/description/urdf/robot/robot.urdf.xacro (robot description, xacro)
@@ -61,25 +61,25 @@
   <xacro:range_sensor
     pos="center"
-    pos_x="0.221"
+    pos_x="${base_length / 2}"
     pos_y="0"
-    pos_z="0.05"
-    roll="0"
+    pos_z="-0.015"
+    pitch="0"
     yaw="0"
   />
   <xacro:range_sensor
     pos="left"
-    pos_x="0.22"
-    pos_y="0.19"
-    pos_z="0.08"
-    roll="1.57"
-    yaw="0.6747"
+    pos_x="${(base_length / 2) - 0.05}"
+    pos_y="0.16"
+    pos_z="-0.015"
+    pitch="0"
+    yaw="0.46364761"
   />
   <xacro:range_sensor
     pos="right"
-    pos_x="0.22"
-    pos_y="-0.19"
-    pos_z="0.08"
-    roll="1.57"
-    yaw="-0.6747"
+    pos_x="${(base_length / 2) - 0.05}"
+    pos_y="-0.16"
+    pos_z="-0.015"
+    pitch="0"
+    yaw="-0.46364761"
   />
   <!-- <xacro:depth_sensor>

File: amrROS2_ws/src/description/urdf/sensors/camera.urdf.xacro (robot description, xacro)
@@ -28,5 +28,5 @@
         <parent link="base_link"/>
         <child link="rgbd_frame" />
-        <origin xyz="0.221 0.0 0.108" rpy="0 -0.6106 0"/>
+        <origin xyz="0.24 0.0 0.12" rpy="0 0 0"/>
       </joint>
       <!-- <gazebo reference="camera">

File: amrROS2_ws/src/description/urdf/sensors/imu.urdf.xacro (robot description, xacro)
@@ -5,5 +5,5 @@
         <parent link="base_link"/>
         <child link="imu_frame"/>
-        <origin xyz="0.178 0 0.075" rpy="0 0 0"/>
+        <origin xyz="0.05 0 0.022" rpy="0 0 0"/>
       </joint>
       <gazebo reference="imu_frame">

File: amrROS2_ws/src/description/urdf/sensors/laser.urdf.xacro (robot description, xacro)
@@ -38,5 +38,5 @@
         <parent link="base_link"/>
         <child link="laser"/>
-        <origin xyz="0.0 0 0.066" rpy="0 0 3.144159265"/>
+        <origin xyz="0.0 0 0.055" rpy="0 0 3.144159265"/>
       </joint>
       <gazebo reference="laser">

File: amrROS2_ws/src/description/urdf/sensors/range_sensor.urdf.xacro (robot description, xacro)
@@ -1,4 +1,4 @@
 <robot xmlns:xacro="http://ros.org/wiki/xacro">
-    <xacro:macro name="range_sensor" params="pos pos_x pos_y pos_z roll yaw">
+    <xacro:macro name="range_sensor" params="pos pos_x pos_y pos_z pitch yaw">
       <link name="${pos}_ranger_link">
         <visual>
@@ -21,5 +21,5 @@
         <parent link="base_link"/>
         <child link="${pos}_ranger_link"/>
-        <origin xyz="${pos_x} ${pos_y} ${pos_z}" rpy="${roll} 0 ${yaw}"/>
+        <origin xyz="${pos_x} ${pos_y} ${pos_z}" rpy="0 ${pitch} ${yaw}"/>
       </joint>
       <gazebo reference="${pos}_ranger_link">
