Commit message: update camera_link module, hardware interface to get and set charging state.

File: amrROS2_ws/src/description/urdf/sensors/camera.urdf.xacro (robot description, xacro)
@@ -1,5 +1,5 @@
 <robot xmlns:xacro="http://ros.org/wiki/xacro">
     <xacro:macro name="camera">
-      <link name="rgbd_frame">
+      <link name="camera_link">
         <visual>
           <origin xyz="0 0 0" rpy="0 0 0"/>
@@ -27,5 +27,5 @@
       <joint name="camera_to_base_link" type="fixed">
         <parent link="base_link"/>
-        <child link="rgbd_frame" />
+        <child link="camera_link" />
         <origin xyz="0.221 0.0 0.108" rpy="0 -0.6106 0"/>
       </joint>
